Commit message: New Models

File: Different Models/drone_description/urdf/drone_description.urdf (robot description, URDF)
Before this commit: robot drone_description, 11 links, 10 joints
Links:
- added link dummy
- link back_arm: mass 0 -> 0.048886
- link drone_body: mass 0.16754 -> 0.16752
Joints:
- added joint dummy_joint: type fixed, parent dummy, child drone_body
- joint back_arm_joint: origin xyz=-0.132701764015227 0 0.0156484811704651 rpy=0 0 0 -> xyz=-0.132701764124662 0 0.0156480902449901 rpy=0 0 0
- joint back_left_prop_joint: axis 0.00321728516721246 0 0.999994824524684 -> 0.0032173 0 0.99999; origin xyz=6.12892824354751E-05 0.1325 0.0190499014071944 rpy=0 0 0 -> xyz=6.1289E-05 0.1325 0.01905 rpy=0 0 0
- joint front_arm_joint: origin xyz=0.132698263984774 0 -0.00435147882953481 rpy=0 0 0 -> xyz=0.132698263875338 0 -0.00435186975500974 rpy=0 0 0
- joint front_left_wing_joint: origin xyz=-3.7249E-05 0.1325 -0.017018 rpy=0 0 0 -> xyz=-3.72493042718469E-05 0.1325 -0.0170179592339789 rpy=0 0 0
- joint front_right_wing_joint: origin xyz=-3.7249E-05 -0.1325 -0.017018 rpy=0 0 0 -> xyz=-3.72493042698485E-05 -0.1325 -0.0170179592339819 rpy=0 0 0

File: test_ws/src/drone_description/urdf/drone_description.urdf (robot description, URDF)
Before this commit: robot drone, 8 links, 7 joints
Links:
- added link back_left_wing, mass 0.010641; collision mesh filename=package://drone_description/meshes/back_left_wing.STL; visual mesh filename=package://drone_description/meshes/back_left_wing.STL
- added link back_right_wing, mass 0.010641; collision mesh filename=package://drone_description/meshes/back_right_wing.STL; visual mesh filename=package://drone_description/meshes/back_right_wing.STL
- added link front_left_wing, mass 0.010641; collision mesh filename=package://drone_description/meshes/front_left_wing.STL; visual mesh filename=package://drone_description/meshes/front_left_wing.STL
- added link front_right_wing, mass 0.010641; collision mesh filename=package://drone_description/meshes/front_right_wing.STL; visual mesh filename=package://drone_description/meshes/front_right_wing.STL
- link back_arm: mass 0.071 -> 0
- link back_left_prop: mass 0.00504005698984341 -> 0.0050401
- link drone_body: mass 0.167539145797033 -> 0.35742
- link front_arm: mass 0.0710004012196545 -> 0.048886
- link front_left_prop: mass 0.00504005698984342 -> 0.0050401
- link front_right_prop: mass 0.00504005698984341 -> 0.0050401
Joints:
- added joint back_left_wing_joint: type fixed, parent back_arm, child back_left_wing, origin xyz=-3.2574E-05 -0.017018 -0.1325 rpy=-1.5708 0 -0.0019141, axis 0 0 0
- added joint back_right_wing_joint: type fixed, parent back_arm, child back_right_wing, origin xyz=-3.2574E-05 -0.017018 0.1325 rpy=-1.5708 0 -0.0019141, axis 0 0 0
- added joint front_left_wing_joint: type fixed, parent front_arm, child front_left_wing, origin xyz=0 -0.017018 -0.1325 rpy=-1.5708 0 6.2965E-05, axis 0 0 0
- added joint front_right_wing_joint: type fixed, parent front_arm, child front_right_wing, origin xyz=0 -0.017018 0.1325 rpy=-1.5708 0 6.2965E-05, axis 0 0 0
- joint back_arm_joint: axis 0 -1 0 -> 0 0 1; origin xyz=-0.1327 0 0.015242 rpy=0 0 0 -> xyz=-0.131247051222321 0.015873762965467 0.014597315603165 rpy=1.5707963267949 0 -0.174532925199433
- joint back_left_prop_joint: axis 0.000709231504572137 0 0.999999748495305 -> 0 0 1; origin xyz=1.35108601620748E-05 0.1325 0.0190499952088355 rpy=0 0 0 -> xyz=3.6463E-05 0.01905 -0.1325 rpy=-1.5708 0 -0.0019141
- joint back_right_prop_joint: axis 0.000709231504572137 0 0.999999748495305 -> 0 0 1; origin xyz=1.35108601621321E-05 -0.1325 0.0190499952088356 rpy=0 0 0 -> xyz=3.64629030858155E-05 0.0190499651038184 0.1325 rpy=-1.5707963267949 0 -0.00191406432285098
- joint front_arm_joint: axis 0 1 0 -> 0 0 -1; origin xyz=0.132700704261176 0 -0.00475833781314276 rpy=0 0 0 -> xyz=0.13275334064868 -0.00722327848964719 -0.00540264439683487 rpy=1.5707963267949 0 0
- joint front_left_prop_joint: axis -0.0020594 0 1 -> 0 0 1; origin xyz=-3.9232E-05 0.1325 0.01905 rpy=0 0 0 -> xyz=0 0.01905 -0.1325 rpy=-1.5708 0 6.2965E-05
- joint front_right_prop_joint: axis -0.00205944392919794 0 0.999997879343103 -> 0 0 1; origin xyz=-3.92324068519967E-05 -0.1325 0.0190499596014851 rpy=0 0 0 -> xyz=0 0.01905 0.1325 rpy=-1.5708 0 6.2965E-05
