Commit message: Added a lot

File: test_ws/src/drone_description/urdf/drone_description.urdf (robot description, URDF)
Before this commit: robot drone, 8 links, 7 joints
Links:
- link back_arm: mass 0.1 -> 0.071
- link back_left_prop: mass 0.02 -> 0.00504005698984341
- link back_right_prop: mass 0.02 -> 0.0050401
- link drone_body: mass .6 -> 0.167539145797033
- link front_arm: mass 0.1 -> 0.0710004012196545
- link front_left_prop: mass 0.02 -> 0.00504005698984342
- link front_right_prop: mass 0.02 -> 0.00504005698984341
Joints:
- joint back_arm_joint: origin xyz=-0.127 0 0 rpy=0 0 0 -> xyz=-0.1327 0 0.015242 rpy=0 0 0
- joint back_left_prop_joint: axis -0.205 0 0.97876 -> 0.000709231504572137 0 0.999999748495305; origin xyz=-0.0013018 0.1524 0.0062151 rpy=0 0 0 -> xyz=1.35108601620748E-05 0.1325 0.0190499952088355 rpy=0 0 0
- joint back_right_prop_joint: axis -0.205 0 0.97876 -> 0.000709231504572137 0 0.999999748495305; origin xyz=-0.0013018 -0.1524 0.0062151 rpy=0 0 0 -> xyz=1.35108601621321E-05 -0.1325 0.0190499952088356 rpy=0 0 0
- joint front_arm_joint: axis 0 -1 0 -> 0 1 0; origin xyz=0.127 0 0 rpy=0 0 0 -> xyz=0.132700704261176 0 -0.00475833781314276 rpy=0 0 0
- joint front_left_prop_joint: axis -0.046167 0 0.99893 -> -0.0020594 0 1; origin xyz=-0.00029316 0.1524 0.0063432 rpy=0 0 0 -> xyz=-3.9232E-05 0.1325 0.01905 rpy=0 0 0
- joint front_right_prop_joint: axis -0.046167 0 0.99893 -> -0.00205944392919794 0 0.999997879343103; origin xyz=-0.00029316 -0.1524 0.0063432 rpy=0 0 0 -> xyz=-3.92324068519967E-05 -0.1325 0.0190499596014851 rpy=0 0 0

Commit message: Adding functionality for wing force

File: test_ws/src/drone_description/urdf/drone_description.urdf (robot description, URDF)
Before this commit: robot drone, 12 links, 11 joints
Links:
- link back_arm: mass 0 -> 0.048886
Joints:
- joint back_left_wing_joint: limit (none) -> lower=-.0001 upper=.0001 effort=100 velocity=.001; type fixed -> revolute
- joint back_right_wing_joint: limit (none) -> lower=-.0001 upper=.0001 effort=100 velocity=.001; type fixed -> prismatic
- joint front_left_wing_joint: limit (none) -> lower=-.0001 upper=.0001 effort=100 velocity=.001; type fixed -> revolute
- joint front_right_wing_joint: limit (none) -> lower=-.0001 upper=.0001 effort=100 velocity=.001; type fixed -> revolute
